File: PixelRing.brd (EAGLE design)
At the start: 36.8 x 36.8 mm, 40 parts, among them Q1 CMA-4544PF-W, SW1 SPST_TACT-KMR2, SW2 SPST_TACT-KMR2, U1 MAX4466EXK+T

Commit message: Add files via upload
Changed micro
Parts:
- removed U$1: PIC18F45K40, 0_Lib_IRSEEM:QFP80P1200X1200X120-44N
- added U2: PIC18F25K22-I/SS, 0_Lib_IRSEEM:SOP65P780X200-28N
- moved SW2 14.1 mm to (23.4, 14.0)
- moved SW1 7.40 mm to (23.4, 19.8)
Connections:
- removed net N$15: SW2.1, SW2.3, U$1.40
- new net N$19: SW2.1, SW2.3, U2.25
- net !MCLR: now also U2.1; no longer U$1.18
- net +5V: now also U2.20; no longer U$1.28, U$1.7
- net GND: now also U2.19, U2.8; no longer U$1.29, U$1.6
- net NEOPIXEL_DI: now also U2.3; no longer U$1.30
- net OUT_MIC: now also U2.2; no longer U$1.36
- net PGC: now also U2.27; no longer U$1.16
- net PGD: now also U2.28; no longer U$1.17
Routing:
- net PGC: track 3.64 -> 15.9 mm, vias 0 -> 1
- net N$19: track 0.00 -> 11.3 mm
- net N$15: track 11.1 -> 0.00 mm
- net PGD: track 2.85 -> 13.9 mm, vias 0 -> 1
- net NEOPIXEL_DI: track 12.3 -> 22.0 mm
- net !MCLR: track 21.2 -> 28.0 mm, vias 2 -> 0
- net +5V: track 18.2 -> 15.0 mm, vias 15 -> 14
- net OUT_MIC: track 11.0 -> 13.5 mm
- net N$16: track 18.5 -> 16.7 mm, vias 2 -> 0
- net GND: track 22.1 -> 22.9 mm
